File: spyrit/kicad_schematic/pyBoard/pyBoard.sch (KiCad schematic (older format))
At the start: 27 parts, among them SW1-RST SPST, Y1 8MHz

Commit message: [Derek] finished pyboard schematic missing only two components, the MIC2005A-1YM5 and the headers
Parts:
- added C16, C17: 2u2, symbol C
- added D1: D_Schottky 1N5819, symbol D_Schottky
- added D2: LED-RED, symbol LED
- added D3: LED-GREEN, symbol LED
- added D4: LED-YELLOW, symbol LED
- added D5: LED-BLUE, symbol LED
- added J9: USB_OTG, symbol USB_OTG
- added R1, R2: 22R, symbol R
- added R10, R16: 560R, symbol R
- added R4, R6, R7: 560, symbol R
- added R8: 220, symbol R
- added R?: R, symbol R
- added SW2-USR: SPST, symbol SPST
- added U2: MCP1754ST-1802E/MB, symbol MCP1754ST-1802E/MB
Connections:
- net +3V3: now also C17.1, U2.3 (VO)
- net GND: now also C16.2, C17.2, D2.1 (K), D3.1 (K), D4.1 (K), D5.1 (K), J9.5 (GND), J9.6 (shield), SW2-USR.1, U2.2 (GND)
- net PA10-ID: now also R1.2
- net PA11-DM: now also R2.2
- net PA12-DP: now also R16.2
- net PA13-RED-P5: now also R4.2
- net PA14-GRN-P4: now also R6.2
- net PA15-YEL-P3: now also R7.2
- net PA9-VBUS: now also R10.2
- net PB3-SW-X17: now also R?.1
- net PB4-BLU-P2: now also R8.2
- new net: D2.2 (A), R4.1
- new net: D3.2 (A), R6.1
- new net: D4.2 (A), R7.1
- new net: J9.2 (D-), R1.1
- new net: J9.3 (D+), R2.1
- new net: J9.4 (ID), R16.1
- new net LED_BLU: D5.2 (A), R8.1
- new net USR-SW: R?.2, SW2-USR.2
- new net VBUS: D1.2 (A), J9.1 (VCC), R10.1
- new net VIN: C16.1, D1.1 (K), U2.1 (VI)
Other:
- note added: "Currently the LED's are not specified to any color"
- note added: "Here is a DNF MIC2005A-1YM5\nUnable to find in the standard KiCAD library\nRefer to PYBv10b for more information"
- note added: "I2C Pullups"
- note added: "In PYBv10b, the MCP1802/3V3\nalso has an EN port"
- note added: "In PYBv10b, this is a four port switch \nwith only two ports being active \nand default to open."
- note added: "in PYBv10b, a CON-USB-MICROAB\nis used with connections: \nVBUS, DM, DP, ID, GND, and MHi lines"
- note removed: "In the original schematic PYBv10b, \nthis is a four port switch with only \ntwo ports being active and default to open."
- moved on the sheet: C1, C10, C13, C19, C2, C20, C3, C4, C5, C6, C8, C9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

Commit message: [Derek] combining the pyboard and the spyrit onto one schematic
Parts:
- added C10p, C3p: 10pF, symbol C
- added C11p: 18pF, symbol C
- added C12p: 8.2pF, symbol C
- added C13p: 1uF, symbol C
- added C14p: 100nF, symbol C
- added C15p: 330pF, symbol C
- added C1p: 100n, symbol C
- added C2p: 12pF, symbol C
- added C4p, C7p, C8p: 220pF, symbol C
- added C5p: 2.2pF, symbol C
- added C6p: 3.3pF, symbol C
- added C9p: 1.8pF, symbol C
- added D1p, D2p, D3p, D4p: LED, symbol LED
- added L10p: 100nH, symbol INDUCTOR
- added L1p: 27nH, symbol INDUCTOR
- added L2p: INDUCTOR, symbol INDUCTOR
- added L3p: 39nH, symbol INDUCTOR
- added L4p, L6p, L9p: 10nH, symbol INDUCTOR
- added L5p: 6.2nH, symbol INDUCTOR
- added L7p: 8.2nH, symbol INDUCTOR
- added L8p: 150nH, symbol INDUCTOR
- added R1p, R2p, R3p, R4p, R5p: R, symbol R
- added U?: SPIRIT1, symbol SPIRIT1
- added Y1p: Crystal, symbol Crystal
Connections:
- net +3V3: now also R1p.1, U?.16 (VBAT), U?.8 (VBAT)
- net GND: now also C10p.1, C11p.1, C12p.1, C13p.1, C14p.1, C15p.1, C1p.1, C2p.2, C3p.2, C5p.2, D1p.1 (K), D2p.1 (K), D3p.1 (K), D4p.1 (K), L1p.1, R5p.2, U?.10 (RFn), U?.11 (GND_PA)
- net PB3-SW-X17: no longer U?.55 (I2S3_CK/SPI1_SCK/SPI3_SCK/SYS_JTDO-SWO/TIM2_CH2/PB3), U?.55 (I2S3_CK/SPI1_SCK/SPI3_SCK/SYS_JTDO-SWO/TIM2_CH2/PB3)
- net PA0-X1: no longer names the net of U?.14 (ADC1_IN0/ADC2_IN0/ADC3_IN0/SYS_WKUP/TIM2_CH1/TIM2_ETR/TIM5_CH1/TIM8_ETR/UART4_TX/USART2_CTS/PA0), U?.14 (ADC1_IN0/ADC2_IN0/ADC3_IN0/SYS_WKUP/TIM2_CH1/TIM2_ETR/TIM5_CH1/TIM8_ETR/UART4_TX/USART2_CTS/PA0)
- net PA1-X2: no longer names the net of U?.15 (ADC1_IN1/ADC2_IN1/ADC3_IN1/TIM2_CH2/TIM5_CH2/UART4_RX/USART2_RTS/PA1), U?.15 (ADC1_IN1/ADC2_IN1/ADC3_IN1/TIM2_CH2/TIM5_CH2/UART4_RX/USART2_RTS/PA1)
- net PA2-X3: no longer names the net of U?.16 (ADC1_IN2/ADC2_IN2/ADC3_IN2/TIM2_CH3/TIM5_CH3/TIM9_CH1/USART2_TX/PA2), U?.16 (ADC1_IN2/ADC2_IN2/ADC3_IN2/TIM2_CH3/TIM5_CH3/TIM9_CH1/USART2_TX/PA2)
- net PA3-X4: no longer names the net of U?.17 (ADC1_IN3/ADC2_IN3/ADC3_IN3/TIM2_CH4/TIM5_CH4/TIM9_CH2/USART2_RX/USB_OTG_HS_ULPI_D0/PA3), U?.17 (ADC1_IN3/ADC2_IN3/ADC3_IN3/TIM2_CH4/TIM5_CH4/TIM9_CH2/USART2_RX/USB_OTG_HS_ULPI_D0/PA3)
- net PA4-X5: no longer names the net of U?.20 (ADC1_IN4/ADC2_IN4/DAC_OUT1/I2S3_WS/SPI1_NSS/SPI3_NSS/USART2_CK/USB_OTG_HS_SOF/PA4), U?.20 (ADC1_IN4/ADC2_IN4/DAC_OUT1/I2S3_WS/SPI1_NSS/SPI3_NSS/USART2_CK/USB_OTG_HS_SOF/PA4)
- net PA5-X6: no longer names the net of U?.21 (ADC1_IN5/ADC2_IN5/DAC_OUT2/SPI1_SCK/TIM2_CH1/TIM2_ETR/TIM8_CH1N/USB_OTG_HS_ULPI_CK/PA5), U?.21 (ADC1_IN5/ADC2_IN5/DAC_OUT2/SPI1_SCK/TIM2_CH1/TIM2_ETR/TIM8_CH1N/USB_OTG_HS_ULPI_CK/PA5)
- net PA6-X7: no longer names the net of U?.22 (ADC1_IN6/ADC2_IN6/SPI1_MISO/TIM13_CH1/TIM1_BKIN/TIM3_CH1/TIM8_BKIN/PA6), U?.22 (ADC1_IN6/ADC2_IN6/SPI1_MISO/TIM13_CH1/TIM1_BKIN/TIM3_CH1/TIM8_BKIN/PA6)
- net PA7-X8: no longer names the net of U?.23 (ADC1_IN7/ADC2_IN7/SPI1_MOSI/TIM14_CH1/TIM1_CH1N/TIM3_CH2/TIM8_CH1N/PA7), U?.23 (ADC1_IN7/ADC2_IN7/SPI1_MOSI/TIM14_CH1/TIM1_CH1N/TIM3_CH2/TIM8_CH1N/PA7)
- net PB0-Y11 renamed PB0-LED_3
- net PB0-LED_3: now also R2p.2
- net PB1-Y12 renamed PB1-SDN
- net PB1-SDN: now also R5p.1, U?.15 (SDN)
- net PB10-Y9 renamed PB10-LED_1
- net PB10-LED_1: now also R4p.2
- net PB11-Y10 renamed PB11-LED_2
- net PB11-LED_2: now also R3p.2
- net PB12-Y5 renamed PB12-CS
- net PB12-CS: now also U?.5 (CSn)
- net PB13-Y6 renamed PB13-SCLK
- net PB13-SCLK: now also U?.4 (SCLK)
- net PB14-Y7 renamed PB14-MISO
- net PB14-MISO: now also U?.2 (MISO)
- net PB15-Y8 renamed PB15-MOSI
- net PB15-MOSI: now also U?.3 (MOSI)
- net PB8-Y3 renamed PB8-GPIO_1
- net PB8-GPIO_1: now also U?.20 (GPIO_1)
- net PB9-Y4 renamed PB9-GPIO_0
- net PB9-GPIO_0: now also U?.1 (GPIO_0)
- net PC0-X19: no longer names the net of U?.8 (PC0/ADC1_IN10/ADC2_IN10/ADC3_IN10/USB_OTG_HS_ULPI_STP), U?.8 (PC0/ADC1_IN10/ADC2_IN10/ADC3_IN10/USB_OTG_HS_ULPI_STP)
- net PC1-X20: no longer names the net of U?.9 (PC1/ADC1_IN11/ADC2_IN11/ADC3_IN11), U?.9 (PC1/ADC1_IN11/ADC2_IN11/ADC3_IN11)
- net PC13-X18: no longer names the net of U?.2 (PC13/ANTI_TAMP/RTC_AF1), U?.2 (PC13/ANTI_TAMP/RTC_AF1)
- net PC2-X21: no longer names the net of U?.10 (PC2/ADC1_IN12/ADC2_IN12/ADC3_IN12/I2S2_ext_SD/SPI2_MISO/USB_OTG_HS_ULPI_DIR), U?.10 (PC2/ADC1_IN12/ADC2_IN12/ADC3_IN12/I2S2_ext_SD/SPI2_MISO/USB_OTG_HS_ULPI_DIR)
- net PC3-X22: no longer names the net of U?.11 (PC3/ADC1_IN13/ADC2_IN13/ADC3_IN13/I2S2_SD/SPI2_MOSI/USB_OTG_HS_ULPI_NXT), U?.11 (PC3/ADC1_IN13/ADC2_IN13/ADC3_IN13/I2S2_SD/SPI2_MOSI/USB_OTG_HS_ULPI_NXT)
- net PC4-X11: no longer names the net of U?.24 (PC4/ADC1_IN14/ADC2_IN14), U?.24 (PC4/ADC1_IN14/ADC2_IN14)
- net PC5-X12: no longer names the net of U?.25 (PC5/ADC1_IN15/ADC2_IN15), U?.25 (PC5/ADC1_IN15/ADC2_IN15)
- net PC6-Y1 renamed PC6-GPIO_3
- net PC6-GPIO_3: now also U?.18 (GPIO_3)
- net PC7-Y2 renamed PC7-GPIO_2
- net PC7-GPIO_2: now also U?.19 (GPIO_2)
- new net: U?.55 (I2S3_CK/SPI1_SCK/SPI3_SCK/SYS_JTDO-SWO/TIM2_CH2/PB3), U?.55 (I2S3_CK/SPI1_SCK/SPI3_SCK/SYS_JTDO-SWO/TIM2_CH2/PB3)
- new net: C5p.1, L2p.2, L3p.1, U?.10 (RFn)
- new net: L7p.2, L8p.1, U?.12 (TX)
- new net: C13p.2, C14p.2, C15p.2, L10p.2, L8p.2, U?.13 (SMPS_ext2)
- new net: L9p.1, U?.14 (SMPS_ext1)
- new net: C1p.2, U?.17 (VREG)
- new net: C2p.1, U?.6 (XOUT), Y1p.1
- new net: C3p.1, U?.7 (XIN), Y1p.2
- new net: C4p.1, C6p.2, L2p.1, U?.9 (RFp)
- new net: D1p.2 (A), R1p.2
- new net: C6p.1, C7p.2, L3p.2
- new net: C4p.2, L1p.2
- new net: C10p.2, C7p.1, C8p.2, C9p.2, L4p.2
- new net: L10p.1, L9p.2
- new net: C12p.2, L6p.1, L7p.1
- new net: C11p.2, L4p.1, L5p.2, L6p.2
- new net: C9p.1, L5p.1
- new net: D2p.2 (A), R2p.1
- new net: D3p.2 (A), R3p.1
- new net: D4p.2 (A), R4p.1
- no-connect marks 9 -> 25
Other:
- note added: "1.0"
- note added: "DR-142-1701-831\ngoes here. Refer to \nIssue #2 on github for\nmore information"
- note added: "FIRECODE Receiver"
- note added: "Here is a DNF MIC2005A-1YM5\nReplacing with the TPS22933A...\nUnable to find in the standard KiCAD library"
- note added: "In Spyrit 992016,\nThis is a four port XTAL\nwith two ports to ground\nNX2016SA-52"
- note added: "MM/DD/YYYY : 10/26/2016"
- note added: "Missing the actual\nSPIRIT-1 component.\nThis is a placeholder only"
- note added: "Ports related to \nunused header pins:\nPC0-PC5, PC13"
- note added: "Ports related to uSD:\nPC8 - PC14, PD2\nThese are no longer required. \nSee FIRECODE documents for\nmore information"
- note added: "Ports related to\nunused header pins:\nPA0-PA7, PB3"
- note added: "There are some\nmissing values\nfrom Spyrit 992016\nthat are required."
- note removed: "Here is a DNF MIC2005A-1YM5\nUnable to find in the standard KiCAD library\nRefer to PYBv10b for more information"
- note removed: "These ports are related to the \nuSD. We have determined that\nthis is not required. See FIRECODE\ndocuments for more information"
- moved on the sheet: C16, C17, D1, D2, D3, D4, D5, J9, R1, R10, R16, R2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
