File: spyrit/kicad_schematic/pyBoard/_saved_pyBoard.sch (KiCad schematic (older format))
At the start: 83 parts, among them J1 USB_OTG, P1 CONN_01X02, SW1-RST1 SPST, SW2-USR1 SPST, U1 MCP1754ST-1802E/MB, U2 SPIRIT1, U3 STM32F405RGTx, U4 TPS22933, Y1 Crystal, Y2 8MHz

Commit message: [Derek] assigning footprints to components, required many elements from github/kicad/
Parts:
- C1, C10, C11, C12, C13, C14, C15, C16, C17, C18, C19, C2, C20, C21, C22, C23, C24, C25, C26, C27, C28, C29, C3, C30, C4, C5, C6, C7, C8, C9: footprint (none) -> Capacitors_SMD:C_0805_HandSoldering
- D1, D1p1, D2, D2p1, D3, D3p1, D4, D4p1: footprint (none) -> LEDs:LED_0805
- D5: footprint (none) -> Diodes_SMD:DD-PAK_TO263_SingleDiode
- J1: footprint (none) -> Connect:USB_Micro-B
- L1, L10, L11, L2, L3, L4, L5, L6, L7, L8, L9: footprint (none) -> Choke_SMD:Choke_SMD_1206_Handsoldering
- P1: footprint (none) -> Socket_Strips:Socket_Strip_Straight_1x02
- R1, R10, R11, R12, R13, R14, R15, R16, R17, R18, R19, R2, R20, R21, R22, R3, R4, R5, R6, R7, R8, R9, R9]1: footprint (none) -> Resistors_SMD:R_0805_HandSoldering
- SW1-RST1, SW2-USR1: footprint (none) -> Buttons_Switches_SMD:SW_SPST_B3S-1100
- U1: footprint (none) -> TO_SOT_Packages_SMD:SOT89-3_Housing_Handsoldering

Commit message: [Derek] wiring intial commit
Parts:
- removed R16, R9]1: 4k7, Resistors_SMD:R_0805_HandSoldering, symbol R
- removed R5: R, Resistors_SMD:R_0805_HandSoldering, symbol R
- removed SW2-USR1: SPST, Buttons_Switches_SMD:SW_SPST_B3S-1100, symbol SPST
- D5: footprint Diodes_SMD:DD-PAK_TO263_SingleDiode -> Diodes_SMD:SMB_Handsoldering
- P1: footprint Socket_Strips:Socket_Strip_Straight_1x02 -> Connect:PINHEAD1-3; symbol CONN_01X02 -> CONN_01X03
- SW1-RST1: footprint Buttons_Switches_SMD:SW_SPST_B3S-1100 -> Buttons_Switches_SMD:SW_SPST_B3U-3000P-B
- U2: footprint (none) -> Housings_DFN_QFN:QFN-20-1EP_4x4mm_Pitch0.5mm
- U3: footprint LQFP64 -> Housings_QFP:LQFP-64_10x10mm_Pitch0.5mm
- U4: footprint (none) -> external_Housings_DFN_QFN:UQFN_1.5mm_x_1.5mm
- Y1, Y2: footprint (none) -> Crystals:Crystal_SMD_5032_2Pads
Connections:
- net RST#: now also P1.3 (P3); no longer C2.1, R1.2, SW1-RST1.1, U3.7 (NRST)
- net at U4.1 (VBAT): now also P1.1 (P1); no longer P1.2 (P2)
- net at U4.3 (DC_IN): now also P1.2 (P2); no longer P1.1 (P1)
- net PB6-SCL-X9: no longer names the net of U3.58 (CAN2_TX/I2C1_SCL/TIM4_CH1/USART1_TX/PB6)
- net PB7-SDA-X10: no longer names the net of U3.59 (I2C1_SDA/TIM4_CH2/USART1_RX/PB7)
- new net: C2.1, R1.2, SW1-RST1.1, U3.7 (NRST)
- no-connect marks 25 -> 27
Other:
- note added: "Ports related to\nunused header pins:\nPA0-PA7, PB3, PB6-PB7"
- note removed: "Ports related to\nunused header pins:\nPA0-PA7, PB3"
- moved on the sheet: C1, C11, C14, C15, C16, C17, C18, C19, C20, C21, C22, C23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
